File: hardware/marsupial.kicad_sch (KiCad schematic)
At the start: 15 parts, among them J101 DC IN, J102 DC OUT, J103 FPC, U101 HT7550-1, U102 XC6206

Commit message: Fix SiC437 footprint and LCSC field error
Parts:
- C101, C102, C103, C104: LCSC ID (none) -> C15849; LCSC Part C15849 -> (none)
- J101, J102: LCSC ID (none) -> C431092
- J103: LCSC ID (none) -> C2856797; LCSC Part C2856797 -> (none)
- U101: LCSC ID (none) -> C16106; LCSC Part C16106 -> (none)
- U102: LCSC ID (none) -> C5446; LCSC Part C5446 -> (none)
Changed lines of the file:
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@@
+			)
+		)
+		(property "LCSC ID" "C431092"
+			(at 265.43 77.47 0)
+			(effects
+				(font
+					(size 1.27 1.27)
+				)
+				(hide yes)
 			)
 		)
@@
 			)
 		)
-		(property "LCSC Part" "C15849"
+		(property "LCSC ID" "C15849"
 			(at 234.95 119.38 0)
 			(effects
@@
 			)
 		)
-		(property "LCSC Part" "C16106"
-			(at 204.47 130.81 0)
+		(property "LCSC ID" "C16106"
+			(at 204.47 113.03 0)
 			(effects
 				(font
@@
 			)
 		)
+		(property "LCSC ID" ""
+			(at 223.52 146.05 0)
+			(effects
+				(font
+					(size 1.27 1.27)
+				)
+				(hide yes)
+			)
+		)
 		(pin "1"
 		)
@@
 			)
 		)
-		(property "LCSC Part" "C15849"
+		(property "LCSC ID" "C15849"
 			(at 189.23 119.38 0)
 			(effects
@@
 			)
 		)
+		(property "LCSC ID" ""
+			(at 241.3 146.05 0)
+			(effects
+				(font
+					(size 1.27 1.27)
+				)
+				(hide yes)
+			)
+		)
 		(pin "1"
 		)
@@
 			)
 		)
+		(property "LCSC ID" "C431092"
+			(at 265.43 44.45 0)
+			(effects
+				(font
+					(size 1.27 1.27)
+				)
+				(hide yes)
+			)
+		)
 		(pin "1"
 		)
@@
 			)
 		)
-		(property "LCSC Part" "C5446"
+		(property "LCSC ID" "C5446"
 			(at 250.19 113.03 0)
 			(effects
@@
 			)
 		)
+		(property "LCSC ID" ""
+			(at 204.47 143.51 0)
+			(effects
+				(font
+					(size 1.27 1.27)
+				)
+				(hide yes)
+			)
+		)
 		(pin "1"
 		)
@@
 			)
 		)
+		(property "LCSC ID" ""
+			(at 250.19 146.05 0)
+			(effects
+				(font
+					(size 1.27 1.27)
+				)
+				(hide yes)
+			)
+		)
 		(pin "1"
 		)
@@
 			)
 		)
-		(property "LCSC Part" "C15849"
+		(property "LCSC ID" "C15849"
 			(at 219.71 119.38 0)
 			(effects
@@
 			)
 		)
+		(property "LCSC ID" ""
+			(at 232.41 146.05 0)
+			(effects
+				(font
+					(size 1.27 1.27)
+				)
+				(hide yes)
+			)
+		)
 		(pin "1"
 		)
@@
 		)
 		(property "Description" "test point"
+			(at 243.84 85.09 0)
+			(effects
+				(font
+					(size 1.27 1.27)
+				)
+				(hide yes)
+			)
+		)
+		(property "LCSC ID" ""
 			(at 243.84 85.09 0)
 			(effects
@@
 			)
 		)
-		(property "LCSC Part" "C15849"
+		(property "LCSC ID" "C15849"
 			(at 265.43 119.38 0)
 			(effects
@@
 			)
 		)
-		(property "LCSC Part" "C2856797"
+		(property "LCSC ID" "C2856797"
 			(at 217.17 78.74 0)
 			(effects
@@
 		)
 		(instances
-			(project "pdcard"
+			(project "marsupial"
 				(path "/a04d6ea3-43ae-48a1-85c5-5c91a24cd719"
 					(page "7")
@@
 		)
 		(instances
-			(project "pdcard"
+			(project "marsupial"
 				(path "/a04d6ea3-43ae-48a1-85c5-5c91a24cd719"
 					(page "5")
@@
 		)
 		(instances
-			(project "pdcard"
+			(project "marsupial"
 				(path "/a04d6ea3-43ae-48a1-85c5-5c91a24cd719"
 					(page "2")
@@
 		)
 		(instances
-			(project "pdcard"
+			(project "marsupial"
 				(path "/a04d6ea3-43ae-48a1-85c5-5c91a24cd719"
 					(page "4")
