File: hardware/usbhub.kicad_sch (KiCad schematic)
At the start: 19 parts, among them J701 USB_C_Receptacle_USB2.0, U701 USB2412-DZK-TR, Y701 24MHz

Commit message: Fix SiC437 footprint and LCSC field error
Parts:
- C701: LCSC ID (none) -> C307331; LCSC Part C307331 -> (none)
- C702, C703: LCSC ID (none) -> C1547; LCSC Part C1547 -> (none)
- C704, C705: LCSC ID (none) -> C14663; LCSC Part C14663 -> (none)
- D701: LCSC ID (none) -> C2290; LCSC Part C2290 -> (none)
- J701: LCSC ID (none) -> C165948; LCSC Part C165948 -> (none)
- R701, R703, R705: LCSC ID (none) -> C25905; LCSC Part C25905 -> (none)
- R702, R704: LCSC ID (none) -> C25744; LCSC Part C25744 -> (none)
- R706: LCSC ID (none) -> C25752; LCSC Part C25752 -> (none)
- R707: LCSC ID (none) -> C138033; LCSC Part C138033 -> (none)
- R708, R709, R710: LCSC ID (none) -> C25794; LCSC Part C25794 -> (none)
- U701: LCSC ID (none) -> C622609; LCSC Part C622609 -> (none)
- Y701: LCSC ID (none) -> C70590; LCSC Part C70590 -> (none)
Changed lines of the file:
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@@
 			)
 		)
-		(property "LCSC Part" "C25744"
+		(property "LCSC ID" "C25744"
 			(at 81.28 77.47 0)
 			(effects
@@
 			)
 		)
-		(property "LCSC Part" "C25794"
+		(property "LCSC ID" "C25794"
 			(at 81.28 113.03 0)
 			(effects
@@
 			)
 		)
-		(property "LCSC Part" "C165948"
+		(property "LCSC ID" "C165948"
 			(at 227.33 86.36 0)
 			(effects
@@
 			)
 		)
-		(property "LCSC Part" "C138033"
+		(property "LCSC ID" "C138033"
 			(at 167.64 100.33 0)
 			(effects
@@
 			)
 		)
-		(property "LCSC Part" "C25905"
+		(property "LCSC ID" "C25905"
 			(at 185.42 71.12 0)
 			(effects
@@
 			)
 		)
-		(property "LCSC Part" "C25752"
+		(property "LCSC ID" "C25752"
 			(at 173.99 91.44 0)
 			(effects
@@
 			)
 		)
-		(property "LCSC Part" "C25905"
+		(property "LCSC ID" "C25905"
 			(at 204.47 78.74 0)
 			(effects
@@
 			)
 		)
-		(property "LCSC Part" "C622609"
-			(at 114.3 127 0)
+		(property "LCSC ID" "C622609"
+			(at 114.3 99.06 0)
 			(effects
 				(font
@@
 			)
 		)
-		(property "LCSC Part" "C1547"
+		(property "LCSC ID" "C1547"
 			(at 185.42 111.76 0)
 			(effects
@@
 			)
 		)
-		(property "LCSC Part" "C25905"
+		(property "LCSC ID" "C25905"
 			(at 204.47 76.2 0)
 			(effects
@@
 			)
 		)
-		(property "LCSC Part" "C1547"
+		(property "LCSC ID" "C1547"
 			(at 173.99 111.76 0)
 			(effects
@@
 			)
 		)
-		(property "LCSC Part" "C70590"
+		(property "LCSC ID" "C70590"
 			(at 194.31 100.33 0)
 			(effects
@@
 			)
 		)
-		(property "LCSC Part" "C2290"
+		(property "LCSC ID" "C2290"
 			(at 72.39 113.03 0)
 			(effects
@@
 			)
 		)
-		(property "LCSC Part" "C307331"
+		(property "LCSC ID" "C307331"
 			(at 71.12 77.47 0)
 			(effects
@@
 			)
 		)
-		(property "LCSC Part" "C25794"
+		(property "LCSC ID" "C25794"
 			(at 157.48 124.46 0)
 			(effects
@@
 			)
 		)
-		(property "LCSC Part" "C25744"
+		(property "LCSC ID" "C25744"
 			(at 176.53 76.2 0)
 			(effects
@@
 			)
 		)
-		(property "LCSC Part" "C25794"
+		(property "LCSC ID" "C25794"
 			(at 148.59 124.46 0)
 			(effects
@@
 			)
 		)
-		(property "LCSC Part" "C14663"
+		(property "LCSC ID" "C14663"
 			(at 81.28 124.46 0)
 			(effects
@@
 			)
 		)
-		(property "LCSC Part" "C14663"
+		(property "LCSC ID" "C14663"
 			(at 167.64 124.46 0)
 			(effects

Commit message: change to C8U3 variant
Parts:
- R707: LCSC ID C138033 -> C26083
